File: Hardware/SparkFun-Blynk-Board-ESP8266.brd (EAGLE design)
At the start: 50 x 41.9 mm, 104 parts, among them IC1 LMV358, Q1 2.5A/30V, Q2 MMBT2222A, Q3 MMBT2222A, U1 MCP73831, U2 ESP8266, U3 AP2112K-3.3V, U4 FT231XS-U, U5 W25Q32FVSS, U6 SI7021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

Commit message: Moving some silk. Updating version number to v10.
Other:
- board text added: "v10"
- board text removed: "v02"
Changed lines of the file:
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@@
 <grid distance="0.05" unitdist="inch" unit="inch" style="lines" multiple="1" display="yes" altdistance="0.005" altunitdist="inch" altunit="inch"/>
 <layers>
-<layer number="1" name="Top" color="4" fill="1" visible="yes" active="yes"/>
+<layer number="1" name="Top" color="4" fill="1" visible="no" active="yes"/>
 <layer number="2" name="Route2" color="1" fill="3" visible="no" active="no"/>
 <layer number="3" name="Route3" color="4" fill="3" visible="no" active="no"/>
@@
 <layer number="19" name="Unrouted" color="6" fill="1" visible="yes" active="yes"/>
 <layer number="20" name="Dimension" color="15" fill="1" visible="yes" active="yes"/>
-<layer number="21" name="tPlace" color="16" fill="1" visible="yes" active="yes"/>
+<layer number="21" name="tPlace" color="16" fill="1" visible="no" active="yes"/>
 <layer number="22" name="bPlace" color="14" fill="1" visible="yes" active="yes"/>
-<layer number="23" name="tOrigins" color="15" fill="1" visible="yes" active="yes"/>
+<layer number="23" name="tOrigins" color="15" fill="1" visible="no" active="yes"/>
 <layer number="24" name="bOrigins" color="15" fill="1" visible="yes" active="yes"/>
 <layer number="25" name="tNames" color="7" fill="1" visible="no" active="yes"/>
@@
 <layer number="47" name="Measures" color="7" fill="1" visible="no" active="yes"/>
 <layer number="48" name="Document" color="7" fill="1" visible="no" active="yes"/>
-<layer number="49" name="Reference" color="7" fill="1" visible="yes" active="yes"/>
+<layer number="49" name="Reference" color="7" fill="1" visible="no" active="yes"/>
 <layer number="50" name="dxf" color="7" fill="1" visible="no" active="no"/>
-<layer number="51" name="tDocu" color="6" fill="1" visible="yes" active="yes"/>
-<layer number="52" name="bDocu" color="7" fill="1" visible="no" active="yes"/>
+<layer number="51" name="tDocu" color="6" fill="1" visible="no" active="yes"/>
+<layer number="52" name="bDocu" color="7" fill="1" visible="yes" active="yes"/>
 <layer number="53" name="tGND_GNDA" color="7" fill="9" visible="no" active="no"/>
 <layer number="54" name="bGND_GNDA" color="1" fill="9" visible="no" active="no"/>
@@
 <wire x1="29.718" y1="34.925" x2="29.972" y2="34.925" width="0.508" layer="21"/>
 <wire x1="29.718" y1="34.925" x2="29.972" y2="34.925" width="0.508" layer="22"/>
-<text x="1.397" y="20.955" size="1.016" layer="16" font="vector" ratio="15" rot="MR90" align="top-center">v02</text>
+<text x="1.397" y="20.955" size="1.016" layer="16" font="vector" ratio="15" rot="MR90" align="top-center">v10</text>
 <text x="2.54" y="27.94" size="0.8128" layer="22" font="vector" ratio="15" rot="MR90" align="bottom-center">GND</text>
 <text x="2.54" y="30.48" size="0.8128" layer="22" font="vector" ratio="15" rot="MR90" align="bottom-center">3V3</text>
@@
 VCC</text>
 <text x="2.54" y="8.255" size="1.016" layer="21" font="vector" ratio="15" rot="R180" align="bottom-center">CHG</text>
-<text x="36.608" y="8.509" size="1.016" layer="22" font="vector" ratio="15" rot="MR90" align="center-right">3.3V</text>
-<text x="40.608" y="8.509" size="1.016" layer="22" font="vector" ratio="15" rot="MR90" align="center-right">DOUT</text>
+<text x="36.608" y="8.509" size="0.8128" layer="22" font="vector" ratio="15" rot="MR90" align="center-right">3.3V</text>
+<text x="40.608" y="8.509" size="0.8128" layer="22" font="vector" ratio="15" rot="MR90" align="center-right">DOUT</text>
 <text x="38.862" y="19.05" size="1.016" layer="21" ratio="15" rot="R180" align="top-center">4</text>
 <text x="13.4239" y="4.826" size="1.016" layer="21" ratio="15" align="bottom-center">3.3V</text>
@@
 <text x="28.6639" y="4.826" size="1.016" layer="21" ratio="15" align="bottom-center">TX</text>
 <text x="33.7439" y="4.826" size="1.016" layer="21" ratio="15" align="bottom-center">5</text>
-<text x="38.608" y="8.509" size="1.016" layer="22" font="vector" ratio="15" rot="MR90" align="center-right">GND</text>
+<text x="38.608" y="8.509" size="0.8128" layer="22" font="vector" ratio="15" rot="MR90" align="center-right">GND</text>
 <text x="8.1661" y="4.826" size="1.016" layer="22" ratio="15" rot="MR0" align="bottom-center">VIN</text>
 <text x="13.2461" y="4.826" size="1.016" layer="22" ratio="15" rot="MR0" align="bottom-center">3.3V</text>
@@
 <text x="31.0261" y="36.8808" size="0.8128" layer="22" ratio="15" rot="MR180" align="bottom-center">RST</text>
 <text x="33.5661" y="37.084" size="1.016" layer="22" ratio="15" rot="MR180" align="bottom-center">0</text>
-<text x="47.625" y="21.59" size="1.27" layer="21" ratio="15" rot="R90" align="top-center">Blynk Board - ESP8266</text>
+<text x="47.752" y="21.082" size="1.3716" layer="21" ratio="15" rot="R90" align="top-center">Blynk Board - ESP8266</text>
 <text x="6.35" y="32.385" size="0.8128" layer="22" font="vector" ratio="15" rot="MR90" align="bottom-center">GND</text>
 <wire x1="3.556" y1="35.56" x2="5.334" y2="34.417" width="0.2032" layer="22"/>
 <wire x1="3.683" y1="30.48" x2="5.334" y2="30.353" width="0.2032" layer="22"/>
 <text x="6.35" y="28.575" size="0.8128" layer="22" font="vector" ratio="15" rot="MR90" align="bottom-center">SDA</text>
-<text x="20.32" y="17.78" size="1.778" layer="22" ratio="15" rot="MR0" align="top-center">Blynk Board - ESP8266</text>
+<text x="21.59" y="17.78" size="1.778" layer="22" ratio="15" rot="MR0" align="top-center">Blynk Board - ESP8266</text>
 </plain>
 <attributes>
